File: Macro_Keyboard_Main_Board_V1.0/Macro_Keyboard_Bottom_V1.0.kicad_pcb (KiCad board)
At the start: 2 copper layers, 130 x 120.1 mm, 88 parts, among them J1 USB_C_Receptacle_USB2.0, J2 JST SM02B-SRSS-TB(LF)(SN), J3 Conn_01x05, Q1 DMG2301L-7, SW1 SW_SPDT PCM12SMTR, SW10 SW_Push, SW11 SW_Push, SW12 SW_Push, SW13 SW_Push, SW14 SW_Push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

Commit message: Newest Changes Added
Other:
- outline, holes or cut-outs redrawn
Changed lines of the file:
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@@
     (fp_line (start 2 7.7) (end 1.5 8.2) (layer "B.SilkS") (width 0.15))
     (fp_arc (start -2.5 6.2) (mid -2.146447 6.346447) (end -2 6.7) (layer "B.SilkS") (width 0.15))
-    (fp_arc (start -1 3.7) (mid -2.06066 3.260659) (end -2.5 2.2) (layer "B.SilkS") (width 0.15))
+    (fp_arc (start -1 3.7) (mid -2.06066 3.26066) (end -2.5 2.2) (layer "B.SilkS") (width 0.15))
     (fp_line (start 7 -7) (end 6 -7) (layer "F.SilkS") (width 0.15))
     (fp_line (start 7 -7) (end 7 -6) (layer "F.SilkS") (width 0.15))
@@
     (fp_line (start -2.5 1.5) (end -7 1.5) (layer "B.Fab") (width 0.15))
     (fp_arc (start -2.5 6.2) (mid -2.146447 6.346447) (end -2 6.7) (layer "B.Fab") (width 0.15))
-    (fp_arc (start -1 3.7) (mid -2.06066 3.260659) (end -2.5 2.2) (layer "B.Fab") (width 0.15))
+    (fp_arc (start -1 3.7) (mid -2.06066 3.26066) (end -2.5 2.2) (layer "B.Fab") (width 0.15))
     (fp_line (start -7.5 -7.5) (end 7.5 -7.5) (layer "F.Fab") (width 0.15))
     (fp_line (start -7.5 7.5) (end -7.5 -7.5) (layer "F.Fab") (width 0.15))
@@
   (gr_line (start 164.1 191) (end 164.09952 105.60048) (layer "Edge.Cuts") (width 0.1))
   (gr_arc (start 164.09952 105.60048) (mid 164.86119 103.761676) (end 166.7 103) (layer "Edge.Cuts") (width 0.1))
-  (gr_line (start 288.95 195.8) (end 267.95 195.8) (layer "Edge.Cuts") (width 0.15))
   (gr_arc (start 169.9 196.2) (mid 222.575044 201.671293) (end 271.6 221.7) (layer "Edge.Cuts") (width 0.1))
   (gr_arc (start 294.1 205.8) (mid 288.921268 218.473813) (end 276 223) (layer "Edge.Cuts") (width 0.1))
   (gr_line (start 294.10048 105.60048) (end 294.1 205.8) (layer "Edge.Cuts") (width 0.1))
   (gr_line (start 166.7 103) (end 291.5 103) (layer "Edge.Cuts") (width 0.1))
-  (gr_line (start 267.95 153.8) (end 267.95 195.8) (layer "Edge.Cuts") (width 0.15))
   (gr_arc (start 291.5 103) (mid 293.338817 103.761663) (end 294.10048 105.60048) (layer "Edge.Cuts") (width 0.1))
   (gr_arc (start 276 223) (mid 273.717202 222.630239) (end 271.6 221.7) (layer "Edge.Cuts") (width 0.1))
-  (gr_line (start 288.95 153.8) (end 288.95 195.8) (layer "Edge.Cuts") (width 0.15))
-  (gr_line (start 267.95 153.8) (end 288.95 153.8) (layer "Edge.Cuts") (width 0.15))
   (gr_circle (center 287.5 109.55) (end 290.5 109.55) (layer "User.1") (width 0.1) (fill none))
   (gr_line (start 167.6 107) (end 228.9 107) (layer "User.1") (width 0.1))
