File: Macro_Keyboard_Main_Board_V1.0/Keyboard.kicad_sch (KiCad schematic)
At the start: 87 parts, among them J1 USB_C_Receptacle_USB2.0, J2 JST SM02B-SRSS-TB(LF)(SN), J3 Conn_01x05, Q1 DMG2301L-7, SW1 SW_SPDT PCM12SMTR, SW10 SW_Push, SW11 SW_Push, SW12 SW_Push, SW13 SW_Push, SW14 SW_Push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

Commit message: Newest Changes Added
Parts:
- SW1: Manufacturer (none) -> C&K; Manufacturer Part Number (none) -> PCM12SMTR
Connections:
- net STAT: now reaches D2.1 (K), U1.1 (STAT)
- net PROG: now reaches R4.1, U1.5 (PROG)
Other:
- note added: "Get some PMV28XPEAR as well"
- moved on the sheet: C2, R4
Changed lines of the file:
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@@
   (junction (at 161.29 26.67) (diameter 0) (color 0 0 0 0)
   )
-  (junction (at 200.025 26.67) (diameter 0) (color 0 0 0 0)
+  (junction (at 190.5 26.67) (diameter 0) (color 0 0 0 0)
   )
   (junction (at 306.07 186.69) (diameter 0) (color 0 0 0 0)
@@
     (stroke (width 0) (type default) (color 0 0 0 0))
   )
-  (wire (pts (xy 184.15 26.67) (xy 200.025 26.67))
+  (wire (pts (xy 184.15 26.67) (xy 190.5 26.67))
     (stroke (width 0) (type default) (color 0 0 0 0))
   )
@@
     (stroke (width 0) (type default) (color 0 0 0 0))
   )
-  (wire (pts (xy 211.455 38.1) (xy 211.455 43.18))
+  (wire (pts (xy 203.2 38.1) (xy 203.2 43.18))
     (stroke (width 0) (type default) (color 0 0 0 0))
   )
@@
     (stroke (width 0) (type default) (color 0 0 0 0))
   )
-  (wire (pts (xy 200.025 26.67) (xy 200.025 29.21))
+  (wire (pts (xy 190.5 26.67) (xy 190.5 29.21))
     (stroke (width 0) (type default) (color 0 0 0 0))
   )
@@
     (stroke (width 0) (type default) (color 0 0 0 0))
   )
-  (wire (pts (xy 218.44 38.1) (xy 211.455 38.1))
+  (wire (pts (xy 218.44 38.1) (xy 203.2 38.1))
     (stroke (width 0) (type default) (color 0 0 0 0))
   )
@@
     (stroke (width 0) (type default) (color 0 0 0 0))
   )
-  (wire (pts (xy 200.025 26.67) (xy 228.6 26.67))
+  (wire (pts (xy 190.5 26.67) (xy 228.6 26.67))
     (stroke (width 0) (type default) (color 0 0 0 0))
   )
@@
     (stroke (width 0) (type default) (color 0 0 0 0))
   )
-  (wire (pts (xy 200.025 36.83) (xy 200.025 39.37))
+  (wire (pts (xy 190.5 36.83) (xy 190.5 39.37))
     (stroke (width 0) (type default) (color 0 0 0 0))
   )
@@
     (stroke (width 0) (type default) (color 0 0 0 0))
   )
-  (wire (pts (xy 211.455 50.8) (xy 211.455 52.07))
+  (wire (pts (xy 203.2 50.8) (xy 203.2 52.07))
     (stroke (width 0) (type default) (color 0 0 0 0))
   )
@@
     (stroke (width 0) (type default) (color 0 0 0 0))
   )
+  (text "Get some PMV28XPEAR as well" (at 298.45 64.77 0)
+    (effects (font (size 1.27 1.27)) (justify left bottom))
+  )
   (text "Power Selector" (at 298.45 49.53 0)
     (effects (font (size 2.54 2.54) (thickness 0.254) bold) (justify left bottom))
@@
     (effects (font (size 2.54 2.54) (thickness 0.254) bold) (justify left bottom))
   )
-  (text "BT Module" (at 88.9 118.745 0)
+  (text "BT Module" (at 111.76 119.38 0)
     (effects (font (size 2.54 2.54) (thickness 0.254) bold) (justify left bottom))
   )
@@
     (effects (font (size 1.27 1.27)) (justify left bottom))
   )
+  (label "PROG" (at 207.01 38.1 0)
+    (effects (font (size 1.27 1.27)) (justify left bottom))
+  )
   (label "ROW2" (at 214.63 175.26 0)
     (effects (font (size 1.27 1.27)) (justify left bottom))
@@
     (effects (font (size 1.27 1.27)) (justify left bottom))
   )
+  (label "STAT" (at 241.3 38.1 0)
+    (effects (font (size 1.27 1.27)) (justify left bottom))
+  )
   (label "COL2" (at 214.63 132.08 0)
     (effects (font (size 1.27 1.27)) (justify left bottom))
@@
       (effects (font (size 1.27 1.27)) hide)
     )
+    (property "Manufacturer" "C&K" (id 4) (at 318.77 71.12 0)
+      (effects (font (size 1.27 1.27)) hide)
+    )
+    (property "Manufacturer Part Number" "PCM12SMTR" (id 5) (at 318.77 71.12 0)
+      (effects (font (size 1.27 1.27)) hide)
+    )
     (pin "1")
     (pin "2")
@@
   )
   (symbol (lib_id "Diode:1N4148W") (at 251.46 146.05 90) (unit 1)
-    (in_bom yes) (on_board yes) (fields_autoplaced)
+    (in_bom yes) (on_board yes)
     (property "Reference" "D5" (id 0) (at 254.635 144.7799 90)
       (effects (font (size 1.27 1.27)) (justify right))
@@
     (pin "2")
   )
-  (symbol (lib_id "power:GND") (at 200.025 39.37 0) (unit 1)
+  (symbol (lib_id "power:GND") (at 190.5 39.37 0) (unit 1)
     (in_bom yes) (on_board yes) (fields_autoplaced)
-    (property "Reference" "#PWR05" (id 0) (at 200.025 45.72 0)
+    (property "Reference" "#PWR05" (id 0) (at 190.5 45.72 0)
       (effects (font (size 1.27 1.27)) hide)
     )
-    (property "Value" "GND" (id 1) (at 200.025 44.45 0))
-    (property "Footprint" "" (id 2) (at 200.025 39.37 0)
+    (property "Value" "GND" (id 1) (at 190.5 44.45 0))
+    (property "Footprint" "" (id 2) (at 190.5 39.37 0)
       (effects (font (size 1.27 1.27)) hide)
     )
-    (property "Datasheet" "" (id 3) (at 200.025 39.37 0)
+    (property "Datasheet" "" (id 3) (at 190.5 39.37 0)
       (effects (font (size 1.27 1.27)) hide)
     )
@@
     (pin "2")
   )
-  (symbol (lib_id "Device:R") (at 211.455 46.99 0) (unit 1)
+  (symbol (lib_id "Device:R") (at 203.2 46.99 0) (unit 1)
     (in_bom yes) (on_board yes) (fields_autoplaced)
-    (property "Reference" "R4" (id 0) (at 213.995 45.7199 0)
+    (property "Reference" "R4" (id 0) (at 205.74 45.7199 0)
       (effects (font (size 1.27 1.27)) (justify left))
     )
-    (property "Value" "20K" (id 1) (at 213.995 48.2599 0)
+    (property "Value" "20K" (id 1) (at 205.74 48.2599 0)
       (effects (font (size 1.27 1.27)) (justify left))
     )
-    (property "Footprint" "Resistor_SMD:R_0603_1608Metric_Pad0.98x0.95mm_HandSolder" (id 2) (at 209.677 46.99 90)
+    (property "Footprint" "Resistor_SMD:R_0603_1608Metric_Pad0.98x0.95mm_HandSolder" (id 2) (at 201.422 46.99 90)
       (effects (font (size 1.27 1.27)) hide)
     )
-    (property "Datasheet" "~" (id 3) (at 211.455 46.99 0)
+    (property "Datasheet" "~" (id 3) (at 203.2 46.99 0)
       (effects (font (size 1.27 1.27)) hide)
     )
-    (property "Size" "0603" (id 4) (at 211.455 46.99 0)
+    (property "Size" "0603" (id 4) (at 203.2 46.99 0)
       (effects (font (size 1.27 1.27)) hide)
     )
@@
     (pin "2")
   )
-  (symbol (lib_id "Device:C") (at 200.025 33.02 0) (unit 1)
+  (symbol (lib_id "Device:C") (at 190.5 33.02 0) (unit 1)
     (in_bom yes) (on_board yes) (fields_autoplaced)
-    (property "Reference" "C2" (id 0) (at 203.835 31.7499 0)
+    (property "Reference" "C2" (id 0) (at 194.31 31.7499 0)
       (effects (font (size 1.27 1.27)) (justify left))
     )
-    (property "Value" "4u7F" (id 1) (at 203.835 34.2899 0)
+    (property "Value" "4u7F" (id 1) (at 194.31 34.2899 0)
       (effects (font (size 1.27 1.27)) (justify left))
     )
-    (property "Footprint" "Capacitor_SMD:C_0603_1608Metric_Pad1.08x0.95mm_HandSolder" (id 2) (at 200.9902 36.83 0)
+    (property "Footprint" "Capacitor_SMD:C_0603_1608Metric_Pad1.08x0.95mm_HandSolder" (id 2) (at 191.4652 36.83 0)
       (effects (font (size 1.27 1.27)) hide)
     )
-    (property "Datasheet" "~" (id 3) (at 200.025 33.02 0))
-    (property "Voltage" "10V" (id 4) (at 200.025 33.02 0)
+    (property "Datasheet" "~" (id 3) (at 190.5 33.02 0))
+    (property "Voltage" "10V" (id 4) (at 190.5 33.02 0)
       (effects (font (size 1.27 1.27)) hide)
     )
-    (property "Size" "0603" (id 5) (at 200.025 33.02 0)
+    (property "Size" "0603" (id 5) (at 190.5 33.02 0)
       (effects (font (size 1.27 1.27)) hide)
     )
@@
     )
   )
-  (symbol (lib_id "power:GND") (at 211.455 52.07 0) (unit 1)
+  (symbol (lib_id "power:GND") (at 203.2 52.07 0) (unit 1)
     (in_bom yes) (on_board yes) (fields_autoplaced)
-    (property "Reference" "#PWR09" (id 0) (at 211.455 58.42 0)
+    (property "Reference" "#PWR09" (id 0) (at 203.2 58.42 0)
       (effects (font (size 1.27 1.27)) hide)
     )
-    (property "Value" "GND" (id 1) (at 211.455 57.15 0))
-    (property "Footprint" "" (id 2) (at 211.455 52.07 0)
+    (property "Value" "GND" (id 1) (at 203.2 57.15 0))
+    (property "Footprint" "" (id 2) (at 203.2 52.07 0)
       (effects (font (size 1.27 1.27)) hide)
     )
-    (property "Datasheet" "" (id 3) (at 211.455 52.07 0)
+    (property "Datasheet" "" (id 3) (at 203.2 52.07 0)
       (effects (font (size 1.27 1.27)) hide)
     )

Commit message: Added notes
Parts:
- R10: value 10K -> 20K
Other:
- note added: "ADD A SMALL BUTTON FOR THE RESET SWITCH."
- note added: "Consider some type of display."
- note added: "FLIPPED SOURCE AND DRAIN"
- note added: "Short the 0R resistor"
- note added: "USB LINES ARE FLIPPED"
- note added: "WRONG CONNECTOR"
- note added: "WRONG FOOTPRINT"
